Commit message: Add files via upload

File: asystr_dual_arm_model/urdf/sherpa.urdf (robot description, URDF)
Before this commit: robot sherpa_dual_arm, 31 links, 30 joints
Links:
- link base_footprint: mass 0.01 -> 15.0
- link base_link: mass None -> 15.0
- link front_left_wheel: mass 0.01 -> 0.2
- link front_left_wheel_base: mass 0.01 -> 0.3
- link front_right_wheel: mass 0.01 -> 0.2
- link front_right_wheel_base: mass 0.01 -> 0.3
- link left_base_link: mass 0.01 -> 2.0
- link left_link_1: mass 0.01 -> 1.0
- link left_link_2: mass 0.01 -> 1.0
- link left_link_3: mass 0.01 -> 1.0
- link left_link_4: mass 0.01 -> 1.0
- link left_link_5: mass 0.01 -> 1.0
- link left_link_6: mass 0.01 -> 1.0
- link left_wrist_adapter: mass 0.01 -> 0.8
- link rear_left_wheel: mass 0.01 -> 0.2
- link rear_left_wheel_base: mass 0.01 -> 0.3
- link rear_right_wheel: mass 0.01 -> 0.2
- link rear_right_wheel_base: mass 0.01 -> 0.3
- link right_base_link: mass 0.01 -> 2.0; geometry collision mesh filename=package://asystr_sensible_model/meshes/collision/asystr_sen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 scale=0.001 0.001 0.001; visual mesh filename=package://asystr_sensible_model/meshes/visual/asystr_sensib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 scale=0.001 0.001 0.001
- link right_link_1: mass 0.01 -> 1.0; geometry collision mesh filename=package://asystr_sensible_model/meshes/collision/asystr_sen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 scale=0.001 0.001 0.001; visual mesh filename=package://asystr_sensible_model/meshes/visual/asystr_sensib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 scale=0.001 0.001 0.001
- link right_link_2: mass 0.01 -> 1.0; geometry collision mesh filename=package://asystr_sensible_model/meshes/collision/asystr_sen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 scale=0.001 0.001 0.001; visual mesh filename=package://asystr_sensible_model/meshes/visual/asystr_sensib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 scale=0.001 0.001 0.001
- link right_link_3: mass 0.01 -> 1.0; geometry collision mesh filename=package://asystr_sensible_model/meshes/collision/asystr_sen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 scale=0.001 0.001 0.001; visual mesh filename=package://asystr_sensible_model/meshes/visual/asystr_sensib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 scale=0.001 0.001 0.001
- link right_link_4: mass 0.01 -> 1.0
- link right_link_5: mass 0.01 -> 1.0; geometry collision box size=0.1 0.1 0.05; visual mesh filename=package://asystr_sensible_model/meshes/visual/RPR/different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 scale=0.001 0.001 0.001
- link right_link_6: mass 0.01 -> 1.0
- link right_wrist_adapter: mass 0.01 -> 0.8
- link sherpa_body: mass 0.01 -> 8.0
- link sherpa_head: mass 0.01 -> 1.0
- link sherpa_head_yaw: mass None -> 2.0
- link telescopic_base: mass 0.01 -> 4.0
- link telescopic_mid: mass 0.01 -> 1.0
Joints:
- joint sherpa_body_joint: limit lower=-0.02 upper=0.47 effort=100.0 velocity=0.1 -> lower=0.0 upper=0.2 effort=50.0 velocity=0.05
- joint telescopic_mid_joint: limit lower=-0.02 upper=0.47 effort=100.0 velocity=0.1 -> lower=0.0 upper=0.2 effort=50.0 velocity=0.05
